File: projects/lights/lights.brd (EAGLE design)
At the start: 100 x 100 mm, 43 parts, among them IC1 LM139DT, IC2 LM139DT, IC3 MCP23017SP

Commit message: lights
Parts:
- added JP1: (no value), pinhead:1X07
- moved FRAME1 87.2 mm to (41.9, 61.0)
- moved D12 12.6 mm to (90.5, 60.3)
- moved D11 12.2 mm to (90.5, 45.1)
- moved D10 11.9 mm to (90.5, 29.8)
- moved D14 9.39 mm to (70.5, 45.1)
- moved D15 9.39 mm to (70.5, 60.3)
- moved S4 8.98 mm to (59.7, 94.0)
- moved S5 8.98 mm to (44.5, 94.0)
- moved S6 8.98 mm to (52.1, 94.0)
- moved VR4 8.89 mm to (90.2, 12.7)
- moved D13 8.86 mm to (70.5, 29.8)
- moved D9 8.56 mm to (50.5, 60.3)
- moved D8 7.97 mm to (50.5, 45.1)
- moved D6 7.65 mm to (30.5, 60.3)
- moved D7 7.56 mm to (50.5, 29.8)
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Connections:
- net !RESET: now also JP1.1
- net GND: now also JP1.4, JP1.5
- net SCL: now also JP1.3
- net SDA: now also JP1.2
- net VDD: now also JP1.6, JP1.7
Routing:
- net VDD: track 0.00 -> 509.6 mm
- net N$19: track 0.00 -> 177.2 mm, vias 0 -> 1
- net N$7: track 0.00 -> 119.6 mm, vias 0 -> 1
- net SCL: track 0.00 -> 110.6 mm
- net SDA: track 0.00 -> 98.0 mm
- net N$18: track 0.00 -> 92.9 mm, vias 0 -> 1
- net N$4: track 0.00 -> 91.8 mm, vias 0 -> 1
- net N$11: track 0.00 -> 89.2 mm, vias 0 -> 1
- net !RESET: track 0.00 -> 88.6 mm
- net N$15: track 0.00 -> 80.1 mm, vias 0 -> 1
- net N$10: track 0.00 -> 65.8 mm
- net N$2: track 0.00 -> 53.1 mm, vias 0 -> 1
- net N$14: track 0.00 -> 44.1 mm
- net N$6: track 0.00 -> 43.9 mm
- net PROX1: track 0.00 -> 40.2 mm, vias 0 -> 1
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- added copper zone on layer 1, net GND
Other:
- board text added: "A0"
- board text added: "A1"
- board text added: "A2"
