File: projects/lights/lights.sch (EAGLE design)
At the start: 43 parts, among them IC1 LM139DT, IC2 LM139DT, IC3 MCP23017SP

Commit message: lights
Parts:
- added JP1: (no value), pinhead:PINHD-1X7
Connections:
- net !RESET: now also JP1.1
- net GND: now also JP1.4, JP1.5
- net SCL: now also JP1.3
- net SDA: now also JP1.2
- net VDD: now also JP1.6, JP1.7
Changed lines of the file:
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@@
 <part name="S5" library="SamacSys_Parts" deviceset="GW22LHP" device=""/>
 <part name="S6" library="SamacSys_Parts" deviceset="GW22LHP" device=""/>
+<part name="JP1" library="pinhead" library_urn="urn:adsk.eagle:library:325" deviceset="PINHD-1X7" device="" package3d_urn="urn:adsk.eagle:package:22477/2"/>
 </parts>
 <sheets>
@@
 <instance part="GND5" gate="1" x="40.64" y="93.98" smashed="yes" rot="MR0">
 <attribute name="VALUE" x="38.1" y="91.186" size="1.778" layer="96" rot="MR0" align="top-center"/>
+</instance>
+<instance part="JP1" gate="A" x="25.4" y="20.32" smashed="yes" rot="R180">
+<attribute name="NAME" x="31.75" y="9.525" size="1.778" layer="95" rot="R180"/>
+<attribute name="VALUE" x="31.75" y="33.02" size="1.778" layer="96" rot="R180"/>
 </instance>
 </instances>
@@
 <label x="76.2" y="99.06" size="1.778" layer="95"/>
 </segment>
+<segment>
+<pinref part="JP1" gate="A" pin="7"/>
+<wire x1="27.94" y1="27.94" x2="58.42" y2="27.94" width="0.1524" layer="91"/>
+<label x="55.88" y="27.94" size="1.778" layer="95"/>
+</segment>
+<segment>
+<pinref part="JP1" gate="A" pin="6"/>
+<wire x1="27.94" y1="25.4" x2="58.42" y2="25.4" width="0.1524" layer="91"/>
+<label x="55.88" y="25.4" size="1.778" layer="95"/>
+</segment>
 </net>
 <net name="N$3" class="0">
@@
 <wire x1="154.94" y1="99.06" x2="162.56" y2="99.06" width="0.1524" layer="91"/>
 <label x="157.48" y="99.06" size="1.778" layer="95"/>
+</segment>
+<segment>
+<pinref part="JP1" gate="A" pin="5"/>
+<wire x1="27.94" y1="22.86" x2="58.42" y2="22.86" width="0.1524" layer="91"/>
+<label x="55.88" y="22.86" size="1.778" layer="95"/>
+</segment>
+<segment>
+<pinref part="JP1" gate="A" pin="4"/>
+<wire x1="27.94" y1="20.32" x2="58.42" y2="20.32" width="0.1524" layer="91"/>
+<label x="55.88" y="20.32" size="1.778" layer="95"/>
 </segment>
 </net>
@@
 </segment>
 </net>
+<net name="SCL" class="0">
+<segment>
+<pinref part="JP1" gate="A" pin="3"/>
+<wire x1="27.94" y1="17.78" x2="58.42" y2="17.78" width="0.1524" layer="91"/>
+<label x="55.88" y="17.78" size="1.778" layer="95"/>
+</segment>
+</net>
+<net name="SDA" class="0">
+<segment>
+<pinref part="JP1" gate="A" pin="2"/>
+<wire x1="27.94" y1="15.24" x2="58.42" y2="15.24" width="0.1524" layer="91"/>
+<label x="55.88" y="15.24" size="1.778" layer="95"/>
+</segment>
+</net>
+<net name="!RESET" class="0">
+<segment>
+<pinref part="JP1" gate="A" pin="1"/>
+<wire x1="27.94" y1="12.7" x2="58.42" y2="12.7" width="0.1524" layer="91"/>
+<label x="55.88" y="12.7" size="1.778" layer="95"/>
+</segment>
+</net>
